File: PCB/picopowered.kicad_pcb (KiCad board)
At the start: 4 copper layers, 21.8 x 52.3 mm, 45 parts, among them J1 Conn_01x20, J2 Conn_01x20, J3 Conn_01x03, P1 USB_C_Plug_USB2.0, Q1 DMG1012T, SW1 BOOTSELECT, SW2 USER_BTN, SW3 RST, U1 RP2040, U2 W25Q32JVSS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

Commit message: Minor Changes
Parts:
- P1: footprint Connector_USB:USB_C_Receptacle_GCT_USB4110 -> Connector_USB:USB_C_Receptacle_HCTL_HC-TYPE-C-16P-01A
Routing:
- net GND: track 25.7 -> 23.6 mm, vias 40 -> 36
